Commit message: test spawn sdf

File: diffdam_description/urdf/diffdam.sec.xacro (robot description, xacro)
@@ -1,9 +1,23 @@
 <?xml version="1.0" ?>
+<!--
+  http://wiki.ros.org/urdf/XML
+  In this xacro file we have defined the following:
+    chasis + caster wheel : link type element
+    wheels : link type elements (left + right)
+    joints : joint type elements (left + right)
+-->
 <robot name="diffdam" xmlns:xacro="https://www.ros.org/wiki/xacro" >
   <xacro:include filename="$(find diffdam_description)/urdf/materials.xacro" />
   <xacro:include filename="$(find diffdam_description)/urdf/diffdam_gazebo.xacro" />
   <xacro:include filename="$(find diffdam_description)/urdf/wheel_macro.xacro" />
+  <!-- Defining link chassis -->
   <link name="link_chassis">
+    <!-- pose and inertial -->
     <pose>0 0 0 0 0 0</pose>
+  <!--
+    All of these elements have some common properties like inertial, collision and visual.
+    The inertial and collision properties enable physics simulation and the visual property controls the appearance of the robot.
+  -->
+    <!-- Inertial properties -->
     <inertial>
       <mass value="5"/>
@@ -11,4 +25,5 @@
       <inertia ixx="0.0395416666667" ixy="0" ixz="0" iyy="0.106208333333" iyz="0" izz="0.106208333333"/>
     </inertial>
+    <!-- Collision properties -->
     <collision name="collision_chassis">
       <geometry>
@@ -16,4 +31,5 @@
       </geometry>
     </collision>
+    <!-- Visual properties -->
     <visual>
       <origin rpy="0 0 0" xyz="0 0 0"/>
@@ -23,4 +39,5 @@
       <material name="white"/>
     </visual>
+    <!-- caster front -->
     <collision name="caster_front_collision">
       <origin rpy=" 0 0 0" xyz="0.2 0 -0.05"/>
@@ -46,13 +63,28 @@
       <material name="white" />
     </visual>
-  </link>
+    </link>
+  <!--
+    Replace the wheel links with the following lines for macros:
+  -->
   <xacro:link_wheel name="link_right_wheel" mass="0.2" length="0.04" radius="0.1"/>
   <xacro:link_wheel name="link_left_wheel" mass="0.2" length="0.04" radius="0.1"/>
+  <!--
+    The joints help in defining the relative motion between links such as the motion of wheel with respect to the chassis. The wheels are links of cylindrical geometry, they are oriented (using rpy property) such that rolling is possible. The placement is controlled via the xyz property. For joints, we have specified the values for damping and friction as well.
+    Both wheels joints are replaced with the following two lines:
+  -->
   <xacro:joint_wheel name="joint_right_wheel"  parent="link_chassis" child="link_right_wheel"  origin_xyz="-0.05 0.15 0"  />
   <xacro:joint_wheel name="joint_left_wheel"   parent="link_chassis" child="link_left_wheel"   origin_xyz="-0.05 -0.15 0"  />
+  <!--
+    Adding a laser scan sensor to the robot
+  -->
   <link name="sensor_laser">
     <inertial>
       <origin xyz="0 0 0" rpy="0 0 0" />
       <mass value="1" />
+      <!-- RANDOM INERTIA BELOW -->
+      <!--
+        OLD INERTIA VALUE - BEFORE RANDOM VALUE INSERTED USING MACROS
+        <inertia ixx="0.02" ixy="0" ixz="0" iyy="0.02" iyz="0" izz="0.02"/>
+      -->
       <xacro:cylinder_inertia mass="1" r="0.05" l="0.1" />
     </inertial>
@@ -98,4 +130,15 @@
     <child link="imu_link"/>
   </joint>
+  <!--
+    Laser gazebo plugin: sensor behaviour to the link
+    Update rate : Controls how often (how fast) the laser data is captured
+    samples : Defines how how many readings are contained in one scan
+    resolution : Defines the minimum angular distance between readings captured in a laser scan
+    range : Defines the minimum sense distance and maximum sense distance. If a point is below minimum sense its reading becomes zero(0) and if a point is further than the maximum sense distance its reading becomes inf. The range resolution defines the minimum distance between 2 points such that two points can be resolved as two separate points.
+    noise : This parameter lets us add gaussian noise to the range data captured by the sensor
+    topicName : Defines the name which is used for publishing the laser data
+    frameName : Defines the link to which the plugin has to be applied
+    see: http://gazebosim.org/tutorials?tut=ros_gzplugins#GPULaser for more information
+  -->
   <gazebo reference="sensor_laser">
     <sensor type="ray" name="head_hokuyo_sensor">
@@ -129,5 +172,5 @@
     </sensor>
   </gazebo>
-  <joint name="camera_joint" type="fixed">
+   <joint name="camera_joint" type="fixed">
     <origin xyz="0.000 0.000 0.2" rpy="0 -1.570796 0"/>
     <parent link="link_chassis"/>
@@ -135,8 +178,9 @@
   </joint>
   <link name="camera_link"/>
-  <gazebo reference="camera_link">
+   <gazebo reference="camera_link">
     <sensor type="camera" name="camera1">
       <update_rate>60.0</update_rate>
       <camera name="fiducial_cam">
+        <!-- <horizontal_fov>1.3962634</horizontal_fov> -->
         <image>
           <width>1080</width>
@@ -150,4 +194,7 @@
         <noise>
           <type>gaussian</type>
+          <!-- Noise is sampled independently per pixel on each frame.
+               That pixel's noise value is added to each of its color
+               channels, which at that point lie in the range [0,1]. -->
           <mean>0.0</mean>
           <stddev>0.007</stddev>
